File: GazSensor/_autosave-GazSensor.kicad_pcb (KiCad board)
At the start: 2 copper layers, 125.5 x 53.5 mm, 21 parts, among them P1 Power, P2 Analog, P3 Digital, P4 Digital, P5 CONN_01X01, P6 CONN_01X01, P7 CONN_01X01, P8 CONN_01X01, U1 LTC1050, U2 RN2483_breakout

Commit message: New sheild
Routing:
- added copper zone on B.Cu, net GND
Changed lines of the file:
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@@
     (mod_text_size 1 1)
     (mod_text_width 0.15)
-    (pad_size 1.6 1.6)
-    (pad_drill 0.8)
+    (pad_size 1.2 1.2)
+    (pad_drill 0.6)
     (pad_to_mask_clearance 0)
     (solder_mask_min_width 0.25)
@@
   (segment (start 120.0785 105.4735) (end 122.7455 102.8065) (width 0.5) (layer B.Cu) (net 45))
   (segment (start 116.1415 105.4735) (end 120.0785 105.4735) (width 0.5) (layer B.Cu) (net 45))
-  (zone (net 0) (net_name "") (layer B.Cu) (hatch edge 0.508)
-    (connect_pads (clearance 0.508))
+  (zone (net 4) (net_name GND) (layer B.Cu) (hatch edge 0.508)
+    (connect_pads yes (clearance 0.508))
     (min_thickness 0.254)
-    (keepout (tracks allowed) (vias allowed) (copperpour not_allowed))
-    (fill (arc_segments 16) (thermal_gap 0.508) (thermal_bridge_width 0.508))
+    (fill yes (arc_segments 16) (thermal_gap 0.508) (thermal_bridge_width 0.508))
     (polygon
       (pts
-        (xy 106.045 68.5165) (xy 105.7275 132.2705) (xy 242.062 134.874) (xy 241.1095 70.485)
+        (xy 102.0445 70.358) (xy 239.7125 70.4215) (xy 238.3155 131.699) (xy 101.346 130.556)
       )
     )
