File: GazSensor/GazSensor.sch (KiCad schematic (older format))
At the start: 21 parts, among them P1 Power, P2 Analog, P3 Digital, P4 Digital, P5 CONN_01X01, P6 CONN_01X01, P7 CONN_01X01, P8 CONN_01X01, U1 LTC1050, U2 RN2483_breakout

Commit message: Rules respected
Parts:
- renumbered RCal2 to RCal1, RCal1 to RCal2
Changed lines of the file:
@@
 encoding utf-8
 Sheet 1 1
-Title "GAZ Sensor qheild"
-Date "lun. 30 mars 2015"
+Title "GAZ Sensor sheild"
+Date "lun. 6 junary 2019"
 Rev ""
 Comp "INSA of Toulouse"
@@
 $EndComp
 $Comp
-L Device:R RCal2
+L Device:R RCal1
 U 1 1 5DFEECEC
 P 3300 2500
-F 0 "RCal2" V 3400 2600 50  0000 R CNN
+F 0 "RCal1" V 3400 2600 50  0000 R CNN
 F 1 "R" V 3200 2550 50  0000 R CNN
 F 2 "Resistor_THT:R_Axial_DIN0207_L6.3mm_D2.5mm_P7.62mm_Horizontal" V 3230 2500 50  0001 C CNN
@@
 	1600 5050 1350 5050
 $Comp
-L Device:R RCal1
+L Device:R RCal2
 U 1 1 5E07BF0B
 P 2750 2500
-F 0 "RCal1" V 2850 2600 50  0000 R CNN
+F 0 "RCal2" V 2850 2600 50  0000 R CNN
 F 1 "R" V 2650 2500 50  0000 R CNN
 F 2 "Resistor_THT:R_Axial_DIN0207_L6.3mm_D2.5mm_P7.62mm_Horizontal" V 2680 2500 50  0001 C CNN
