File: GazSensor/GazSensor.sch (KiCad schematic (older format))
At the start: 23 parts, among them J101 Conn_01x03, J102 Conn_01x03, P1 Power, P2 Analog, P3 Digital, P4 Digital, P5 CONN_01X01, P6 CONN_01X01, P7 CONN_01X01, P8 CONN_01X01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

Commit message: Image of last sheild
Parts:
- J101, J102: footprint (none) -> Connector_PinHeader_2.00mm:PinHeader_1x03_P2.00mm_Vertical
Other:
- moved on the sheet: U2
Changed lines of the file:
@@
 L power:GND #PWR0101
 U 1 1 5DFE3C4A
-P 9600 4200
-F 0 "#PWR0101" H 9600 3950 50  0001 C CNN
-F 1 "GND" H 9605 4027 50  0000 C CNN
-F 2 "" H 9600 4200 50  0001 C CNN
-F 3 "" H 9600 4200 50  0001 C CNN
-	1    9600 4200
+P 1350 1300
+F 0 "#PWR0101" H 1350 1050 50  0001 C CNN
+F 1 "GND" H 1355 1127 50  0000 C CNN
+F 2 "" H 1350 1300 50  0001 C CNN
+F 3 "" H 1350 1300 50  0001 C CNN
+	1    1350 1300
 	1    0    0    -1
 $EndComp
@@
 L power:+5V #PWR0103
 U 1 1 5DFE3CEB
-P 10250 4200
-F 0 "#PWR0103" H 10250 4050 50  0001 C CNN
-F 1 "+5V" H 10265 4373 50  0000 C CNN
-F 2 "" H 10250 4200 50  0001 C CNN
-F 3 "" H 10250 4200 50  0001 C CNN
-	1    10250 4200
+P 2000 1300
+F 0 "#PWR0103" H 2000 1150 50  0001 C CNN
+F 1 "+5V" H 2015 1473 50  0000 C CNN
+F 2 "" H 2000 1300 50  0001 C CNN
+F 3 "" H 2000 1300 50  0001 C CNN
+	1    2000 1300
 	-1   0    0    1
 $EndComp
@@
 L power:PWR_FLAG #FLG0102
 U 1 1 5DFE3E0C
-P 10250 4200
-F 0 "#FLG0102" H 10250 4275 50  0001 C CNN
-F 1 "PWR_FLAG" H 10250 4374 50  0000 C CNN
-F 2 "" H 10250 4200 50  0001 C CNN
-F 3 "~" H 10250 4200 50  0001 C CNN
-	1    10250 4200
+P 2000 1300
+F 0 "#FLG0102" H 2000 1375 50  0001 C CNN
+F 1 "PWR_FLAG" H 2000 1474 50  0000 C CNN
+F 2 "" H 2000 1300 50  0001 C CNN
+F 3 "~" H 2000 1300 50  0001 C CNN
+	1    2000 1300
 	1    0    0    -1
 $EndComp
@@
 L power:PWR_FLAG #FLG0101
 U 1 1 5DFE3E5E
-P 9600 4200
-F 0 "#FLG0101" H 9600 4275 50  0001 C CNN
-F 1 "PWR_FLAG" H 9600 4374 50  0000 C CNN
-F 2 "" H 9600 4200 50  0001 C CNN
-F 3 "~" H 9600 4200 50  0001 C CNN
-	1    9600 4200
+P 1350 1300
+F 0 "#FLG0101" H 1350 1375 50  0001 C CNN
+F 1 "PWR_FLAG" H 1350 1474 50  0000 C CNN
+F 2 "" H 1350 1300 50  0001 C CNN
+F 3 "~" H 1350 1300 50  0001 C CNN
+	1    1350 1300
 	1    0    0    -1
 $EndComp
@@
 L GazSensor-rescue:RN2483_breakout-MyComponents U2
 U 1 1 5DFE64BC
-P 7950 3850
-F 0 "U2" H 8528 3515 50  0000 L CNN
-F 1 "RN2483_breakout" H 8528 3424 50  0000 L CNN
-F 2 "MyComponents:RN2483_Breakout" H 7950 3850 50  0001 C CNN
-F 3 "" H 7950 3850 50  0001 C CNN
-	1    7950 3850
-	1    0    0    -1
-$EndComp
-NoConn ~ 7650 4450
-NoConn ~ 7800 4450
-NoConn ~ 8250 4450
+P 2100 1600
+F 0 "U2" H 2678 1265 50  0000 L CNN
+F 1 "RN2483_breakout" H 2678 1174 50  0000 L CNN
+F 2 "MyComponents:RN2483_Breakout" H 2100 1600 50  0001 C CNN
+F 3 "" H 2100 1600 50  0001 C CNN
+	1    2100 1600
+	1    0    0    -1
+$EndComp
+NoConn ~ 1800 2200
+NoConn ~ 1950 2200
+NoConn ~ 2400 2200
 $Comp
 L Device:R R6
@@
 Wire Wire Line
 	7750 3100 7750 2950
-Text Label 7350 4600 0    60   ~ 0
+Text Label 1500 2350 0    60   ~ 0
 7
-Text Label 7500 4600 0    60   ~ 0
+Text Label 1650 2350 0    60   ~ 0
 8
 $Comp
 L power:GND #PWR0110
 U 1 1 5DFF6303
-P 8400 4450
-F 0 "#PWR0110" H 8400 4200 50  0001 C CNN
-F 1 "GND" H 8405 4277 50  0000 C CNN
-F 2 "" H 8400 4450 50  0001 C CNN
-F 3 "" H 8400 4450 50  0001 C CNN
-	1    8400 4450
+P 2550 2200
+F 0 "#PWR0110" H 2550 1950 50  0001 C CNN
+F 1 "GND" H 2555 2027 50  0000 C CNN
+F 2 "" H 2550 2200 50  0001 C CNN
+F 3 "" H 2550 2200 50  0001 C CNN
+	1    2550 2200
 	1    0    0    -1
 $EndComp
@@
 L power:+3.3V #PWR0109
 U 1 1 5DFF64C3
-P 8100 4450
-F 0 "#PWR0109" H 8100 4300 50  0001 C CNN
-F 1 "+3.3V" H 8100 4600 50  0000 C CNN
-F 2 "" H 8100 4450 50  0000 C CNN
-F 3 "" H 8100 4450 50  0000 C CNN
-	1    8100 4450
+P 2250 2200
+F 0 "#PWR0109" H 2250 2050 50  0001 C CNN
+F 1 "+3.3V" H 2250 2350 50  0000 C CNN
+F 2 "" H 2250 2200 50  0000 C CNN
+F 3 "" H 2250 2200 50  0000 C CNN
+	1    2250 2200
 	-1   0    0    1
 $EndComp
-Text Label 7950 4700 0    60   ~ 0
+Text Label 2100 2450 0    60   ~ 0
 Reset
 Wire Wire Line
-	7350 4450 7350 4600
-Wire Wire Line
-	7500 4450 7500 4600
-Wire Wire Line
-	7950 4450 7950 4700
+	1500 2200 1500 2350
+Wire Wire Line
+	1650 2200 1650 2350
+Wire Wire Line
+	2100 2200 2100 2450
 Wire Wire Line
 	5950 2350 6500 2350
@@
 L power:PWR_FLAG #FLG0103
 U 1 1 5E00A427
-P 10750 4200
-F 0 "#FLG0103" H 10750 4275 50  0001 C CNN
-F 1 "PWR_FLAG" H 10750 4374 50  0000 C CNN
-F 2 "" H 10750 4200 50  0001 C CNN
-F 3 "~" H 10750 4200 50  0001 C CNN
-	1    10750 4200
+P 2500 1300
+F 0 "#FLG0103" H 2500 1375 50  0001 C CNN
+F 1 "PWR_FLAG" H 2500 1474 50  0000 C CNN
+F 2 "" H 2500 1300 50  0001 C CNN
+F 3 "~" H 2500 1300 50  0001 C CNN
+	1    2500 1300
 	1    0    0    -1
 $EndComp
@@
 L power:+3.3V #PWR0113
 U 1 1 5E00A4AC
-P 10750 4200
-F 0 "#PWR0113" H 10750 4050 50  0001 C CNN
-F 1 "+3.3V" H 10765 4373 50  0000 C CNN
-F 2 "" H 10750 4200 50  0001 C CNN
-F 3 "" H 10750 4200 50  0001 C CNN
-	1    10750 4200
+P 2500 1300
+F 0 "#PWR0113" H 2500 1150 50  0001 C CNN
+F 1 "+3.3V" H 2515 1473 50  0000 C CNN
+F 2 "" H 2500 1300 50  0001 C CNN
+F 3 "" H 2500 1300 50  0001 C CNN
+	1    2500 1300
 	-1   0    0    1
 $EndComp
@@
 F 0 "J102" V 4900 5450 50  0000 L CNN
 F 1 "Conn_01x03" V 5000 5100 50  0000 L CNN
-F 2 "" H 4900 5250 50  0001 C CNN
+F 2 "Connector_PinHeader_2.00mm:PinHeader_1x03_P2.00mm_Vertical" H 4900 5250 50  0001 C CNN
 F 3 "~" H 4900 5250 50  0001 C CNN
 	1    4900 5250
@@
 F 0 "J101" V 4773 5030 50  0000 L CNN
 F 1 "Conn_01x03" V 4864 5030 50  0000 L CNN
-F 2 "" H 4900 4850 50  0001 C CNN
+F 2 "Connector_PinHeader_2.00mm:PinHeader_1x03_P2.00mm_Vertical" H 4900 4850 50  0001 C CNN
 F 3 "~" H 4900 4850 50  0001 C CNN
 	1    4900 4850

Commit message: Last Commit
Parts:
- removed U1: LTC1050, MyComponents:PDIP-8_N, symbol MyComponents:LTC1050
- removed U101: GazSensor, Package_TO_SOT_THT:TO-5-10_Window, symbol GazSensor-rescue:GazSensor
- removed U2: RN2483_breakout, MyComponents:RN2483_Breakout, symbol GazSensor-rescue:RN2483_breakout-MyComponents
- added U101: RN2483_breakout, MyComponents:RN2483_Breakout, symbol RN2483_breakout:RN2483_breakout
- added U102: GazSensor, Package_TO_SOT_THT:TO-5-10_Window, symbol GazSensorLib:GazSensor
- added U103: LTC1050, MyComponents:LTC1050, symbol LTC1050:LTC1050
Connections:
- wire segments 91 -> 89
Changed lines of the file:
@@
 	0    1    1    0
-$EndComp
-$Comp
-L GazSensor-rescue:RN2483_breakout-MyComponents U2
-U 1 1 5DFE64BC
-P 2100 1600
-F 0 "U2" H 2678 1265 50  0000 L CNN
-F 1 "RN2483_breakout" H 2678 1174 50  0000 L CNN
-F 2 "MyComponents:RN2483_Breakout" H 2100 1600 50  0001 C CNN
-F 3 "" H 2100 1600 50  0001 C CNN
-	1    2100 1600
-	1    0    0    -1
 $EndComp
 NoConn ~ 1800 2200
@@
 NoConn ~ 10550 1300
 NoConn ~ 9400 3000
-$Comp
-L MyComponents:LTC1050 U1
-U 1 1 5E044E85
-P 5500 2400
-F 0 "U1" H 5400 2150 50  0000 C CNN
-F 1 "LTC1050" H 5100 2150 50  0000 C CNN
-F 2 "MyComponents:PDIP-8_N" H 5500 2400 50  0001 C CNN
-F 3 "" H 5500 2400 50  0001 C CNN
-	1    5500 2400
-	1    0    0    -1
-$EndComp
 NoConn ~ 6000 2800
 NoConn ~ 4400 2800
@@
 Wire Wire Line
 	6500 3050 6000 3050
-Wire Wire Line
-	3950 3050 4400 3050
 Wire Wire Line
 	3950 750  3950 3050
@@
 Wire Wire Line
 	2900 750  2600 750
-Wire Wire Line
-	3400 3300 4400 3300
-$Comp
-L GazSensor-rescue:GazSensor U101
-U 1 1 5E23ADB2
-P 2000 4300
-F 0 "U101" H 2400 4325 50  0000 C CNN
-F 1 "GazSensor" H 2400 4234 50  0000 C CNN
-F 2 "Package_TO_SOT_THT:TO-5-10_Window" H 2000 4300 50  0001 C CNN
-F 3 "" H 2000 4300 50  0001 C CNN
-	1    2000 4300
-	1    0    0    -1
-$EndComp
 $Comp
 L power:GND #PWR0114
@@
 	0    -1   -1   0
 $EndComp
-$Comp
-L power:+5V #PWR0116
-U 1 1 5E240BAC
-P 3350 4450
-F 0 "#PWR0116" H 3350 4300 50  0001 C CNN
-F 1 "+5V" H 3365 4623 50  0000 C CNN
-F 2 "" H 3350 4450 50  0001 C CNN
-F 3 "" H 3350 4450 50  0001 C CNN
-	1    3350 4450
-	1    0    0    -1
-$EndComp
-Wire Wire Line
-	3350 4450 3350 4500
-Wire Wire Line
-	3350 4500 3150 4500
 $Comp
 L Connector_Generic:Conn_01x03 J102
@@
 Text Label 5800 4350 2    50   ~ 0
 linkCircuit
-$Comp
-L power:+5V #PWR0102
-U 1 1 5E2D648D
+Wire Wire Line
+	5750 5700 4900 5700
+Wire Wire Line
+	2400 3300 1600 3300
+$Comp
+L power:+3.3V #PWR0102
+U 1 1 5E245755
 P 5750 5700
 F 0 "#PWR0102" H 5750 5550 50  0001 C CNN
-F 1 "+5V" V 5765 5828 50  0000 L CNN
+F 1 "+3.3V" V 5765 5828 50  0000 L CNN
 F 2 "" H 5750 5700 50  0001 C CNN
 F 3 "" H 5750 5700 50  0001 C CNN
@@
 	0    1    1    0
 $EndComp
-Wire Wire Line
-	5750 5700 4900 5700
-Wire Wire Line
-	2400 3300 1600 3300
+$Comp
+L power:+5V #PWR0116
+U 1 1 5E248F8E
+P 3150 4500
+F 0 "#PWR0116" H 3150 4350 50  0001 C CNN
+F 1 "+5V" H 3165 4673 50  0000 C CNN
+F 2 "" H 3150 4500 50  0001 C CNN
+F 3 "" H 3150 4500 50  0001 C CNN
+	1    3150 4500
+	1    0    0    -1
+$EndComp
+Wire Wire Line
+	3400 3300 4400 3300
+Wire Wire Line
+	3950 3050 4400 3050
+$Comp
+L GazSensorLib:GazSensor U102
+U 1 1 5E273C63
+P 2250 4200
+F 0 "U102" H 2400 4125 50  0000 C CNN
+F 1 "GazSensor" H 2400 4034 50  0000 C CNN
+F 2 "Package_TO_SOT_THT:TO-5-10_Window" H 2250 4200 50  0001 C CNN
+F 3 "" H 2250 4200 50  0001 C CNN
+	1    2250 4200
+	1    0    0    -1
+$EndComp
+$Comp
+L RN2483_breakout:RN2483_breakout U101
+U 1 1 5E277401
+P 2100 1600
+F 0 "U101" H 2678 1265 50  0000 L CNN
+F 1 "RN2483_breakout" H 2678 1174 50  0000 L CNN
+F 2 "MyComponents:RN2483_Breakout" H 2100 1600 50  0001 C CNN
+F 3 "" H 2100 1600 50  0001 C CNN
+	1    2100 1600
+	1    0    0    -1
+$EndComp
+$Comp
+L LTC1050:LTC1050 U103
+U 1 1 5E27AAB2
+P 5500 2400
+F 0 "U103" H 5200 2815 50  0000 C CNN
+F 1 "LTC1050" H 5200 2724 50  0000 C CNN
+F 2 "MyComponents:LTC1050" H 5500 2400 50  0001 C CNN
+F 3 "" H 5500 2400 50  0001 C CNN
+	1    5500 2400
+	1    0    0    -1
+$EndComp
 $EndSCHEMATC

Commit message: Last kicad version
Parts:
- added R101: R, Resistor_THT:R_Axial_DIN0207_L6.3mm_D2.5mm_P7.62mm_Horizontal, symbol Device:R
- U103: footprint MyComponents:LTC1050 -> Package_DIP:DIP-8_W7.62mm_LongPads
Connections:
- net +5V: no longer U102.3 (HeartSensor)
- net A0: now also U102.6 (TempSensor), R101.1
- net GND: now also R101.2; no longer U102.8 (HeartSensor)
- no-connect marks 36 -> 34
Changed lines of the file:
@@
 EESchema Schematic File Version 4
-LIBS:GazSensor-cache
 EELAYER 26 0
 EELAYER END
@@
 	9150 1900 9150 1450
 Wire Wire Line
-	9400 2500 8900 2500
-Wire Wire Line
 	9400 2600 8900 2600
 Wire Wire Line
@@
 	2600 5450 2650 5450
 $Comp
-L power:GND #PWR0115
-U 1 1 5E240ADC
-P 3150 4600
-F 0 "#PWR0115" H 3150 4350 50  0001 C CNN
-F 1 "GND" V 3155 4472 50  0000 R CNN
-F 2 "" H 3150 4600 50  0001 C CNN
-F 3 "" H 3150 4600 50  0001 C CNN
-	1    3150 4600
-	0    -1   -1   0
-$EndComp
-$Comp
 L Connector_Generic:Conn_01x03 J102
 U 1 1 5E24510F
@@
 	0    -1   -1   0
 $EndComp
-NoConn ~ 1650 4500
-NoConn ~ 1650 4600
 Text Label 850  4800 0    50   ~ 0
 GazSensorLeft_Pin7
@@
 	0    1    1    0
 $EndComp
-$Comp
-L power:+5V #PWR0116
-U 1 1 5E248F8E
-P 3150 4500
-F 0 "#PWR0116" H 3150 4350 50  0001 C CNN
-F 1 "+5V" H 3165 4673 50  0000 C CNN
-F 2 "" H 3150 4500 50  0001 C CNN
-F 3 "" H 3150 4500 50  0001 C CNN
-	1    3150 4500
-	1    0    0    -1
-$EndComp
 Wire Wire Line
 	3400 3300 4400 3300
@@
 U 1 1 5E27AAB2
 P 5500 2400
-F 0 "U103" H 5200 2815 50  0000 C CNN
-F 1 "LTC1050" H 5200 2724 50  0000 C CNN
-F 2 "MyComponents:LTC1050" H 5500 2400 50  0001 C CNN
+F 0 "U103" H 5200 2200 50  0000 C CNN
+F 1 "LTC1050" H 5250 2300 50  0000 C CNN
+F 2 "Package_DIP:DIP-8_W7.62mm_LongPads" H 5500 2400 50  0001 C CNN
 F 3 "" H 5500 2400 50  0001 C CNN
 	1    5500 2400
 	1    0    0    -1
 $EndComp
+Wire Wire Line
+	9400 2500 8550 2500
+Wire Wire Line
+	8550 1400 8550 2500
+Wire Wire Line
+	7700 1400 8150 1400
+Text Label 7700 1400 0    50   ~ 0
+TempSensor
+$Comp
+L Device:R R101
+U 1 1 5E28B7B2
+P 8150 1700
+F 0 "R101" H 8220 1746 50  0000 L CNN
+F 1 "R" H 8220 1655 50  0000 L CNN
+F 2 "Resistor_THT:R_Axial_DIN0207_L6.3mm_D2.5mm_P7.62mm_Horizontal" V 8080 1700 50  0001 C CNN
+F 3 "~" H 8150 1700 50  0001 C CNN
+	1    8150 1700
+	1    0    0    -1
+$EndComp
+$Comp
+L power:GND #PWR0115
+U 1 1 5E28B8B1
+P 8150 2000
+F 0 "#PWR0115" H 8150 1750 50  0001 C CNN
+F 1 "GND" H 8155 1827 50  0000 C CNN
+F 2 "" H 8150 2000 50  0001 C CNN
+F 3 "" H 8150 2000 50  0001 C CNN
+	1    8150 2000
+	1    0    0    -1
+$EndComp
+Wire Wire Line
+	8150 2000 8150 1850
+Wire Wire Line
+	8150 1550 8150 1400
+Connection ~ 8150 1400
+Wire Wire Line
+	8150 1400 8550 1400
+Wire Wire Line
+	1650 4600 850  4600
+Text Label 850  4600 0    50   ~ 0
+TempSensor
 $EndSCHEMATC
