File: GazSensor/_saved_GazSensor.sch (KiCad schematic (older format))
At the start: 23 parts, among them J101 Conn_01x03, J102 Conn_01x03, P1 Power, P2 Analog, P3 Digital, P4 Digital, P5 CONN_01X01, P6 CONN_01X01, P7 CONN_01X01, P8 CONN_01X01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

Commit message: Last Version with Aime Gaz Sensor
Parts:
- J101, J102: footprint (none) -> Connector_PinHeader_2.00mm:PinHeader_1x03_P2.00mm_Vertical
Changed lines of the file:
@@
 F 0 "J102" V 4900 5450 50  0000 L CNN
 F 1 "Conn_01x03" V 5000 5100 50  0000 L CNN
-F 2 "" H 4900 5250 50  0001 C CNN
+F 2 "Connector_PinHeader_2.00mm:PinHeader_1x03_P2.00mm_Vertical" H 4900 5250 50  0001 C CNN
 F 3 "~" H 4900 5250 50  0001 C CNN
 	1    4900 5250
@@
 F 0 "J101" V 4773 5030 50  0000 L CNN
 F 1 "Conn_01x03" V 4864 5030 50  0000 L CNN
-F 2 "" H 4900 4850 50  0001 C CNN
+F 2 "Connector_PinHeader_2.00mm:PinHeader_1x03_P2.00mm_Vertical" H 4900 4850 50  0001 C CNN
 F 3 "~" H 4900 4850 50  0001 C CNN
 	1    4900 4850
