File: GazSensor/GazSensor.kicad_pcb (KiCad board)
At the start: 2 copper layers, 128.3 x 53.3 mm, 20 parts, among them P1 Power, P2 Analog, P3 Digital, P4 Digital, P5 CONN_01X01, P6 CONN_01X01, P7 CONN_01X01, P8 CONN_01X01, U101 RN2483_breakout, U102 LTC1050

Commit message: New sheild
Parts:
- removed C101, C103, C104: 100n, Capacitor_THT:C_Radial_D4.0mm_H5.0mm_P1.50mm
- removed C102: 1u, Capacitor_THT:C_Radial_D4.0mm_H5.0mm_P1.50mm
- removed R101: 10k, Resistor_THT:R_Axial_DIN0207_L6.3mm_D2.5mm_P7.62mm_Horizontal
- removed R102, R104: 100k, Resistor_THT:R_Axial_DIN0207_L6.3mm_D2.5mm_P7.62mm_Horizontal
- removed R103, R105: 1k, Resistor_THT:R_Axial_DIN0207_L6.3mm_D2.5mm_P7.62mm_Horizontal
- removed RGazSensor101: R, MyComponents:GazSensor
- removed U101: RN2483_breakout, MyComponents:RN2483_Breakout
- removed U102: LTC1050, MyComponents:PDIP-8_N
- added C1: 100n, Capacitor_THT:CP_Radial_D4.0mm_P1.50mm, F.Cu at (124.2, 88.8)
- added C2: 100n, Capacitor_THT:CP_Radial_D4.0mm_P1.50mm, F.Cu at (167.8, 112.5)
- added C3: 1u, Capacitor_THT:CP_Radial_D4.0mm_P1.50mm, F.Cu at (149.5, 91.7)
- added C4: 1u, Capacitor_THT:CP_Radial_D4.0mm_P1.50mm, F.Cu at (133.8, 113.3)
- added R1: 100k, Resistor_THT:R_Axial_DIN0207_L6.3mm_D2.5mm_P7.62mm_Horizontal, F.Cu at (133.3, 91.4)
- added R3: 100k, Resistor_THT:R_Axial_DIN0207_L6.3mm_D2.5mm_P7.62mm_Horizontal, F.Cu at (129.3, 123.4)
- added R5: 10k, Resistor_THT:R_Axial_DIN0207_L6.3mm_D2.5mm_P7.62mm_Horizontal, F.Cu at (148.7, 83.6)
- added R6: 1k, Resistor_THT:R_Axial_DIN0207_L6.3mm_D2.5mm_P7.62mm_Horizontal, F.Cu at (168.0, 101.7)
- added RCal1: R, Resistor_THT:R_Axial_DIN0207_L6.3mm_D2.5mm_P7.62mm_Horizontal, F.Cu at (122.7, 102.8)
- added RCal2: R, Resistor_THT:R_Axial_DIN0207_L6.3mm_D2.5mm_P7.62mm_Horizontal, F.Cu at (116.1, 113.1)
- added RSensor101: R, MyComponents:GazSensor, F.Cu at (162.7, 87.5)
- added U1: LTC1050, MyComponents:PDIP-8_N, F.Cu at (147.7, 105.0)
- added U2: RN2483_breakout, MyComponents:RN2483_Breakout, F.Cu at (187.8, 88.0)
Routing:
- net GND: track 191.8 -> 0.00 mm
- net /A0: track 184.2 -> 25.3 mm
- net Net-(C101-Pad1): track 89.3 -> 0.00 mm
- net Net-(C103-Pad2): track 79.3 -> 0.00 mm
- net +3V3: track 78.1 -> 154.0 mm
- net Net-(C103-Pad1): track 50.5 -> 0.00 mm
- net Net-(C4-Pad2): track 0.00 -> 42.5 mm
- net Net-(C4-Pad1): track 0.00 -> 40.7 mm
- net /Reset: track 70.8 -> 101.5 mm
- net Net-(C1-Pad1): track 0.00 -> 19.7 mm
- net Net-(R101-Pad1): track 18.8 -> 0.00 mm
- net Net-(R5-Pad1): track 0.00 -> 12.0 mm
- net +5V: track 43.7 -> 51.9 mm
- net Net-(RCal1-Pad1): track 0.00 -> 7.71 mm
- net /8: track 45.7 -> 41.3 mm
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- added copper zone on B.Cu, net GND
Other:
- board size 128.3 x 53.3 mm -> 125.5 x 53.5 mm
- rule trace_min: 0.1 -> 0.2
- board text added: "Sheild V.Laurens_M.Commérot_H.Safri"
- board text removed: "Gaz Sensor Sheild -Background) (LaurensV, Commérot, Safri)"
- board text removed: "Gaz Sensor Sheild( Foreground) (LaurensV, Commérot, Safri)"

Commit message: Rules respected
Parts:
- moved C2 2.71 mm to (165.2, 111.6), turned to 0 degrees
Routing:
- net GND: track 0.00 -> 146.3 mm, vias 0 -> 6
- net /7: track 39.3 -> 43.3 mm
- net /Reset: track 101.5 -> 104.9 mm
- net +3V3: track 154.0 -> 155.2 mm
- net /8: track 41.3 -> 42.3 mm
- removed copper zone on B.Cu, net GND
Other:
- board outline removed
- net class Default: clearance 0.2 -> 0.4; trace_width 0.25 -> 0.8; via_dia 0.6 -> 1.6; via_drill 0.4 -> 0.8
- net class Power added: clearance 0.4, trace_width 1, via_dia 1.6, via_drill 0.8
- rule trace_clearance: 0.2 -> 0.4

Commit message: PCB Good
Routing:
- net GND: track 146.3 -> 0.00 mm, vias 6 -> 0
- added copper zone on B.Cu, net GND

Commit message: Last Version with Aime Gaz Sensor
Parts:
- removed RSensor101: R, MyComponents:GazSensor
- added J101: Conn_01x03, Connector_PinHeader_2.00mm:PinHeader_1x03_P2.00mm_Vertical, F.Cu at (155.6, 83.2)
- added J102: Conn_01x03, Connector_PinHeader_2.00mm:PinHeader_1x03_P2.00mm_Vertical, F.Cu at (169.9, 96.6)
- added U101: GazSensor, Package_TO_SOT_THT:TO-5-10_Window, F.Cu at (163.7, 86.6)
Connections:
- R5 pad 1: Net-(R5-Pad1) -> /linkCircuit
Routing:
- net +3V3: track 155.2 -> 87.4 mm
- net /GazSensorLeft_Pin9: track 0.00 -> 17.8 mm
- net /GazSensorLeft_Pin7: track 0.00 -> 15.8 mm
- net +5V: track 51.5 -> 67.1 mm
- net Net-(R5-Pad1): track 12.0 -> 0.00 mm
- net /GazSensorRight_Pin2: track 0.00 -> 9.16 mm
- net /GazSensorRight_Pin4: track 0.00 -> 8.25 mm
- net /linkCircuit: track 0.00 -> 7.53 mm
- net /Reset: track 104.9 -> 101.9 mm
- net /8: track 42.3 -> 41.4 mm

Commit message: Last Commit
Parts:
- removed U1: LTC1050, MyComponents:PDIP-8_N
- removed U101: GazSensor, Package_TO_SOT_THT:TO-5-10_Window
- added U102: GazSensor, Package_TO_SOT_THT:TO-5-10_Window, F.Cu at (163.7, 86.6)
- added U103: LTC1050, MyComponents:LTC1050, F.Cu at (147.6, 105.0)
Connections:
- J102 pad 2: +5V -> +3V3
Routing:
- net +3V3: track 87.4 -> 109.4 mm
- net +5V: track 67.1 -> 62.3 mm

Commit message: Last kicad version
Parts:
- removed U2: RN2483_breakout, MyComponents:RN2483_Breakout
- added R101: R, Resistor_THT:R_Axial_DIN0207_L6.3mm_D2.5mm_P7.62mm_Horizontal, F.Cu at (165.1, 118.7)
- added U101: RN2483_breakout, MyComponents:RN2483_Breakout, F.Cu at (187.8, 88.0)
- U103: footprint MyComponents:LTC1050 -> Package_DIP:DIP-8_W7.62mm
- moved U103 10.7 mm to (140.1, 97.3)
Connections:
- U102 pad 3: +5V -> Net-(U102-Pad3)
- U102 pad 6: Net-(U102-Pad6) -> /A0
- U102 pad 8: GND -> Net-(U102-Pad8)
Routing:
- net +5V: track 62.3 -> 51.5 mm
- net /A0: track 25.5 -> 28.8 mm
