File: OldVersion/GazSensor/GazSensor.kicad_pcb (KiCad board)
At the start: 2 copper layers, 23 parts, among them J101 Conn_01x03, J102 Conn_01x03, P1 Power, P2 Analog, P3 Digital, P4 Digital, P5 CONN_01X01, P6 CONN_01X01, P7 CONN_01X01, P8 CONN_01X01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

Commit message: Last Version with Aime Gaz Sensor
Parts:
- removed J101, J102: Conn_01x03, Connector_PinHeader_2.00mm:PinHeader_1x03_P2.00mm_Vertical
- removed U101: GazSensor, Package_TO_SOT_THT:TO-5-10_Window
- added RSensor101: R, MyComponents:GazSensor, F.Cu at (162.7, 87.5)
Connections:
- R5 pad 1: /linkCircuit -> Net-(R5-Pad1)
Routing:
- net +3V3: track 87.4 -> 155.2 mm
- net /GazSensorLeft_Pin9: track 17.8 -> 0.00 mm
- net /GazSensorLeft_Pin7: track 15.8 -> 0.00 mm
- net +5V: track 67.1 -> 51.5 mm
- net Net-(R5-Pad1): track 0.00 -> 12.0 mm
- net /GazSensorRight_Pin2: track 9.16 -> 0.00 mm
- net /GazSensorRight_Pin4: track 8.25 -> 0.00 mm
- net /linkCircuit: track 7.53 -> 0.00 mm
- net /Reset: track 101.9 -> 104.9 mm
- net /8: track 41.4 -> 42.3 mm
